Commit message: driving through Gazebo

File: description/robot.urdf.xacro (robot description, xacro)
@@ -2,3 +2,4 @@
 <robot xmlns:xacro="http://www.ros.org/wiki/xacro"  name="ilios">
    <xacro:include filename="robot_core.xacro" />
+   <xacro:include filename="gazebo_control.xacro" />
 </robot>

File: description/robot_core.xacro (robot description, xacro)
@@ -42,4 +42,7 @@
     </collision>
 </link>
+<gazebo reference="chassis">
+    <material>Gazebo/White</material>
+</gazebo>
 <!-- LEFT WHEEL -->
 <joint name="left_wheel_joint" type="continuous">
@@ -65,4 +68,7 @@
     </xacro:inertial_cylinder>
 </link>
+<gazebo reference="left_wheel">
+    <material>Gazebo/blue</material>
+</gazebo>
 <!-- RIGHT WHEEL -->
 <joint name="right_wheel_joint" type="continuous">
@@ -83,9 +89,12 @@
             <cylinder length="0.04" radius="0.05" />
         </geometry>
-        <xacro:inertial_cylinder mass="0.1" length="0.05" radius="0.05">
+    </collision>
+    <xacro:inertial_cylinder mass="0.1" length="0.05" radius="0.05">
         <origin xyz="0 0 0" rpy="0 0 0"/>
     </xacro:inertial_cylinder>
-    </collision>
 </link>
+<gazebo reference="right_wheel">
+    <material>Gazebo/blue</material>
+</gazebo>
 <!-- CASTER WHEEL -->
 <joint name="caster_wheel_joint" type="fixed">
@@ -110,3 +119,8 @@
     </xacro:inertial_sphere>
 </link>
+<gazebo reference="caster_wheel">
+    <material>Gazebo/black</material>
+    <mu1 value="0.001"/>
+    <mu2 value="0.001"/>
+</gazebo>
 </robot>

Commit message: till LIDAR

File: description/robot.urdf.xacro (robot description, xacro)
@@ -3,3 +3,4 @@
    <xacro:include filename="robot_core.xacro" />
    <xacro:include filename="gazebo_control.xacro" />
+   <xacro:include filename="lidar.xacro" />
 </robot>

File: description/robot_core.xacro (robot description, xacro)
@@ -7,5 +7,5 @@
 </material>
 <material name="orange">
-    <color rgba="1 0.3 0.1 1"/>
+     <color rgba="${255/255} ${108/255} ${10/255} 1.0"/>
 </material>
 <material name="blue">
@@ -15,4 +15,10 @@
     <color rgba="0 0 0 1"/>
 </material>
+<material name="red">
+    <color rgba="1 0 0 1"/>
+</material>
+  <material name="yellow">
+      <color rgba="1 1 0 1"/>
+    </material>
 <!-- BASE LINK -->
 <link name="base_link">
@@ -26,17 +32,17 @@
 <link name="chassis">
     <visual>
-        <origin xyz="0.15 0 0.075" rpy="0 0 0"/>
+        <origin xyz="0.075 0 0.035" rpy="0 0 0"/>
         <geometry>
-            <box size="0.3 0.3 0.15"/>
+            <box size="0.2 0.15 0.07"/>
         </geometry>
-        <material name="white"/>
+        <material name="orange"/>
     </visual>
     <collision>
          <origin xyz="0.15 0 0.075" rpy="0 0 0"/>
         <geometry>
-            <box size="0.3 0.3 0.15"/>
+            <box size="0.2 0.15 0.07"/>
         </geometry>
-        <xacro:inertial_box mass="0.5" x="0.3" y="0.3" z="0.15">
-        <origin xyz="0.15 0 0.075" rpy="0 0 0"/>
+        <xacro:inertial_box mass="0.5" x="0.2" y="0.15" z="0.07">
+        <origin xyz="0.2 0 0.07" rpy="0 0 0"/>
     </xacro:inertial_box>
     </collision>
@@ -47,7 +53,7 @@
 <!-- LEFT WHEEL -->
 <joint name="left_wheel_joint" type="continuous">
-    <parent link="base_link"/>
+    <parent link="chassis"/>
     <child link="left_wheel"/>
-    <origin xyz="0 0.175 0" rpy="-${pi/2} 0 0"/>
+    <origin xyz="0.07 0.08 0" rpy="-${pi/2} 0 0"/>
     <axis xyz="0 0 1"/>
 </joint>
@@ -55,14 +61,14 @@
     <visual>
         <geometry>
-            <cylinder length="0.04" radius="0.05" />
+            <cylinder length="0.03" radius="0.03" />
         </geometry>
-        <material name="blue"/>
+        <material name="yellow"/>
     </visual>
     <collision>
          <geometry>
-            <cylinder length="0.04" radius="0.05" />
+            <cylinder length="0.03" radius="0.03" />
         </geometry>
     </collision>
-    <xacro:inertial_cylinder mass="0.1" length="0.05" radius="0.05">
+    <xacro:inertial_cylinder mass="0.1" length="0.03" radius="0.03">
         <origin xyz="0 0 0" rpy="0 0 0"/>
     </xacro:inertial_cylinder>
@@ -73,7 +79,7 @@
 <!-- RIGHT WHEEL -->
 <joint name="right_wheel_joint" type="continuous">
-    <parent link="base_link"/>
+    <parent link="chassis"/>
     <child link="right_wheel"/>
-    <origin xyz="0 -0.175 0" rpy="${pi/2} 0 0"/>
+    <origin xyz="0.07 -0.08 0" rpy="${pi/2} 0 0"/>
     <axis xyz="0 0 -1"/>
 </joint>
@@ -81,14 +87,14 @@
     <visual>
         <geometry>
-            <cylinder length="0.04" radius="0.05" />
+            <cylinder length="0.03" radius="0.03" />
         </geometry>
-        <material name="blue"/>
+        <material name="yellow"/>
     </visual>
     <collision>
         <geometry>
-            <cylinder length="0.04" radius="0.05" />
+            <cylinder length="0.03" radius="0.03" />
         </geometry>
     </collision>
-    <xacro:inertial_cylinder mass="0.1" length="0.05" radius="0.05">
+    <xacro:inertial_cylinder mass="0.1" length="0.03" radius="0.03">
         <origin xyz="0 0 0" rpy="0 0 0"/>
     </xacro:inertial_cylinder>
@@ -101,19 +107,19 @@
     <parent link="chassis"/>
     <child link="caster_wheel"/>
-    <origin xyz="0.24 0 0" rpy="0 0 0"/>
+    <origin xyz="0.15 0 0" rpy="0 0 0"/>
 </joint>
 <link name="caster_wheel">
     <visual>
         <geometry>
-            <sphere radius="0.05" />
+            <sphere radius="0.02" />
         </geometry>
-        <material name="black"/>
+        <material name="white"/>
     </visual>
     <collision>
         <geometry>
-            <sphere radius="0.05" />
+            <sphere radius="0.02" />
         </geometry>
     </collision>
-    <xacro:inertial_sphere mass="0.1" radius="0.05">
+    <xacro:inertial_sphere mass="0.1" radius="0.02">
         <origin xyz="0 0 0" rpy="0 0 0"/>
     </xacro:inertial_sphere>
